File: testing-split-kb/testing-split-kb.kicad_pcb (KiCad board)
At the start: 2 copper layers, 121.5 x 73.1 mm, 37 parts, among them J1 Conn_01x08_Pin, SW1 SW_Push_Dual, SW10 SW_Push_Dual, SW11 SW_Push_Dual, SW12 SW_Push_Dual, SW13 SW_Push_Dual, SW14 SW_Push_Dual, SW15 SW_Push_Dual, SW2 SW_Push_Dual, SW3 SW_Push_Dual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

Commit message: WIP
Parts:
- removed REF**: TestPoint_Plated_Hole_D2.0mm, TestPoint:TestPoint_Plated_Hole_D2.0mm
- added ?: , , F.Cu at (77.0, 37.0)
- J1: value Conn_01x08_Pin -> Conn_01x09_Pin; footprint Connector_PinHeader_2.54mm:PinHeader_1x08_P2.54mm_Vertical -> Connector_PinHeader_2.54mm:PinHeader_1x09_P2.54mm_Vertical
- moved D5 1.70 mm to (170.0, 37.3)
- moved D1 1.70 mm to (94.2, 37.1)
- moved D2 1.70 mm to (113.0, 37.1)
- moved D3 1.70 mm to (131.6, 37.1)
- moved D4 1.70 mm to (150.8, 37.2)
Routing:
- net row2: track 289.7 -> 308.2 mm
- net row3: track 199.5 -> 215.8 mm
- net row1: track 127.9 -> 133.1 mm
- net Net-(D1-A): track 25.8 -> 29.2 mm
- net col5: track 225.5 -> 227.4 mm
- net col1: track 202.9 -> 204.3 mm
- net col4: track 230.1 -> 230.9 mm
- net Net-(D5-A): track 22.7 -> 23.5 mm
- net Net-(D3-A): track 22.6 -> 23.3 mm
- net Net-(D4-A): track 22.6 -> 23.4 mm
- added copper zone on In1.Cu, net GND
- added copper zone on In2.Cu, net GND
Other:
- copper layers 2 -> 4
- board text added: "GND"
- board text added: "Testing key matrix v1.1"
- board text removed: "Testing key matrix v1.0"
