File: testing-split-kb/testing-split-kb.kicad_sch (KiCad schematic)
At the start: 31 parts, among them J1 Conn_01x08_Pin, SW1 SW_Push_Dual, SW10 SW_Push_Dual, SW11 SW_Push_Dual, SW12 SW_Push_Dual, SW13 SW_Push_Dual, SW14 SW_Push_Dual, SW15 SW_Push_Dual, SW2 SW_Push_Dual, SW3 SW_Push_Dual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

Commit message: WIP
Parts:
- D1, D10, D11, D12, D13, D14, D15, D2, D3, D4, D5, D6, D7, D8, D9: footprint Diode_THT:D_DO-35_SOD27_P7.62mm_Horizontal -> TestingSplitKb:D_DO-35_SOD27_P7.62mm_Horizontal_BothSides
- J1: value Conn_01x08_Pin -> Conn_01x09_Pin; footprint Connector_PinHeader_2.54mm:PinHeader_1x08_P2.54mm_Vertical -> Connector_PinHeader_2.54mm:PinHeader_1x09_P2.54mm_Vertical; symbol Connector:Conn_01x08_Pin -> Connector:Conn_01x09_Pin
Connections:
- new net GND: J1.9 (Pin_9)
